File: 16-relays.kicad_sch (KiCad schematic)
At the start: 120 parts, among them J1 Conn_01x12_Socket, J2 Conn_01x12_Socket, J3 POWER, K1 AHQSH112LM100G, K10 AHQSH112LM100G, K11 AHQSH112LM100G, K12 AHQSH112LM100G, K13 AHQSH112LM100G, K14 AHQSH112LM100G, K15 AHQSH112LM100G, K16 AHQSH112LM100G, K2 AHQSH112LM100G, K3 AHQSH112LM100G, K4 AHQSH112LM100G, K5 AHQSH112LM100G, K6 AHQSH112LM100G, K7 AHQSH112LM100G, K8 AHQSH112LM100G, K9 AHQSH112LM100G, Q1 2N7000, Q10 2N7000, Q11 2N7000, Q12 2N7000, Q13 2N7000, Q14 2N7000, Q15 2N7000, Q16 2N7000, Q2 2N7000, Q3 2N7000, Q4 2N7000, Q5 2N7000, Q6 2N7000, Q7 2N7000, Q8 2N7000, Q9 2N7000, SW1 Mode Button, U1 PicoW, U3 L7805

Commit message: Update 16-relays.kicad_sch
adjust LED current limiting resistors
Parts:
- R22, R23, R24, R25, R26, R27, R28, R29, R30, R31, R32, R33, R34, R35, R36, R37: value 330 -> 1K
Changed lines of the file:
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@@
 			)
 		)
-		(property "Value" "330"
+		(property "Value" "1K"
 			(at 253.1872 185.293 0)
 			(effects
@@
 			)
 		)
-		(property "Value" "330"
+		(property "Value" "1K"
 			(at 253.1872 246.253 0)
 			(effects
@@
 			)
 		)
-		(property "Value" "330"
+		(property "Value" "1K"
 			(at 169.3672 246.253 0)
 			(effects
@@
 			)
 		)
-		(property "Value" "330"
+		(property "Value" "1K"
 			(at 253.1872 35.433 0)
 			(effects
@@
 			)
 		)
-		(property "Value" "330"
+		(property "Value" "1K"
 			(at 169.3672 215.773 0)
 			(effects
@@
 			)
 		)
-		(property "Value" "330"
+		(property "Value" "1K"
 			(at 253.1872 156.083 0)
 			(effects
@@
 			)
 		)
-		(property "Value" "330"
+		(property "Value" "1K"
 			(at 169.3672 126.873 0)
 			(effects
@@
 			)
 		)
-		(property "Value" "330"
+		(property "Value" "1K"
 			(at 253.1872 126.873 0)
 			(effects
@@
 			)
 		)
-		(property "Value" "330"
+		(property "Value" "1K"
 			(at 169.3672 65.913 0)
 			(effects
@@
 			)
 		)
-		(property "Value" "330"
+		(property "Value" "1K"
 			(at 253.1872 96.393 0)
 			(effects
@@
 			)
 		)
-		(property "Value" "330"
+		(property "Value" "1K"
 			(at 169.3672 185.293 0)
 			(effects
@@
 			)
 		)
-		(property "Value" "330"
+		(property "Value" "1K"
 			(at 169.3672 96.393 0)
 			(effects
@@
 			)
 		)
-		(property "Value" "330"
+		(property "Value" "1K"
 			(at 253.1872 65.913 0)
 			(effects
@@
 			)
 		)
-		(property "Value" "330"
+		(property "Value" "1K"
 			(at 253.1872 215.773 0)
 			(effects
@@
 			)
 		)
-		(property "Value" "330"
+		(property "Value" "1K"
 			(at 169.3672 35.433 0)
 			(effects
@@
 			)
 		)
-		(property "Value" "330"
+		(property "Value" "1K"
 			(at 169.3672 156.083 0)
 			(effects
