File: 16-relays.kicad_pcb (KiCad board)
At the start: 2 copper layers, 184.7 x 104.7 mm, 122 parts, among them J1 Conn_01x12_Socket, J2 Conn_01x12_Socket, J3 POWER, K1 AHQSH112LM100G, K10 AHQSH112LM100G, K11 AHQSH112LM100G, K12 AHQSH112LM100G, K13 AHQSH112LM100G, K14 AHQSH112LM100G, K15 AHQSH112LM100G, K16 AHQSH112LM100G, K2 AHQSH112LM100G, K3 AHQSH112LM100G, K4 AHQSH112LM100G, K5 AHQSH112LM100G, K6 AHQSH112LM100G, K7 AHQSH112LM100G, K8 AHQSH112LM100G, K9 AHQSH112LM100G, Q1 2N7000, Q10 2N7000, Q11 2N7000, Q12 2N7000, Q13 2N7000, Q14 2N7000, Q15 2N7000, Q16 2N7000, Q2 2N7000, Q3 2N7000, Q4 2N7000, Q5 2N7000, Q6 2N7000, Q7 2N7000, Q8 2N7000, Q9 2N7000, SW1 Mode Button, U1 PicoW, U3 L7805

Commit message: add doc
Parts:
- added G***: LOGO, parts:non-ionizing-bigger, F.Cu at (58.0, 79.0)
Changed lines of the file:
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@@
+		)
+	)
+	(footprint "parts:non-ionizing-bigger"
+		(layer "F.Cu")
+		(at 58 79)
+		(property "Reference" "G***"
+			(at 0 0 0)
+			(layer "F.SilkS")
+			(hide yes)
+			(effects
+				(font
+					(size 1.524 1.524)
+					(thickness 0.3)
+				)
+			)
+		)
+		(property "Value" "LOGO"
+			(at 0.75 0 0)
+			(layer "F.SilkS")
+			(hide yes)
+			(effects
+				(font
+					(size 1.524 1.524)
+					(thickness 0.3)
+				)
+			)
+		)
+		(property "Footprint" "parts:non-ionizing-bigger"
+			(at 0 0 0)
+			(layer "F.Fab")
+			(hide yes)
+			(effects
+				(font
+					(size 1.27 1.27)
+					(thickness 0.15)
+				)
+			)
+		)
+		(property "Datasheet" ""
+			(at 0 0 0)
+			(layer "F.Fab")
+			(hide yes)
+			(effects
+				(font
+					(size 1.27 1.27)
+					(thickness 0.15)
+				)
+			)
+		)
+		(property "Description" ""
+			(at 0 0 0)
+			(layer "F.Fab")
+			(hide yes)
+			(effects
+				(font
+					(size 1.27 1.27)
+					(thickness 0.15)
+				)
+			)
+		)
+		(attr through_hole)
+		(fp_poly
+			(pts
+				(xy 0.239931 -1.133503) (xy 0.300902 -1.087685) (xy 0.410841 -0.970749) (xy 0.453275 -0.839761)
+				(xy 0.4572 -0.755176) (xy 0.415481 -0.542704) (xy 0.296572 -0.39266) (xy 0.109837 -0.314269) (xy 0 -0.3048)
+				(xy -0.183442 -0.330641) (xy -0.322535 -0.419736) (xy -0.33251 -0.429491) (xy -0.438007 -0.600263)
+				(xy -0.459681 -0.796796) (xy -0.397969 -0.988081) (xy -0.323273 -1.085273) (xy -0.148882 -1.197644)
+				(xy 0.043674 -1.213739) (xy 0.239931 -1.133503)
+			)
+			(stroke
+				(width 0.01)
+				(type solid)
+			)
+			(fill solid)
+			(layer "F.SilkS")
+		)
+		(fp_poly
+			(pts
+				(xy -1.06534 -1.802079) (xy -0.998617 -1.725745) (xy -1.008856 -1.66328) (xy -1.03507 -1.630055)
+				(xy -1.215279 -1.351242) (xy -1.315732 -1.031928) (xy -1.336858 -0.694001) (xy -1.279088 -0.35935)
+				(xy -1.142854 -0.049864) (xy -1.000234 0.140954) (xy -0.894332 0.256509) (xy -1.107534 0.469711)
+				(xy -1.290374 0.222155) (xy -1.482894 -0.116745) (xy -1.590397 -0.484473) (xy -1.613099 -0.862503)
+				(xy -1.551213 -1.232311) (xy -1.404956 -1.575369) (xy -1.267262 -1.772224) (xy -1.192321 -1.852397)
+				(xy -1.137621 -1.858868) (xy -1.06534 -1.802079)
+			)
+			(stroke
+				(width 0.01)
+				(type solid)
+			)
+			(fill solid)
+			(layer "F.SilkS")
+		)
+		(fp_poly
+			(pts
+				(xy -1.923869 -2.65447) (xy -1.884736 -2.620848) (xy -1.831812 -2.566454) (xy -1.820924 -2.515154)
+				(xy -1.858598 -2.439932) (xy -1.95136 -2.313773) (xy -1.962426 -2.299269) (xy -2.226331 -1.875303)
+				(xy -2.400301 -1.421441) (xy -2.484316 -0.950833) (xy -2.478357 -0.476628) (xy -2.382404 -0.011974)
+				(xy -2.196437 0.429981) (xy -1.967069 0.778617) (xy -1.814058 0.973034) (xy -1.915755 1.074732)
+				(xy -2.017453 1.17643) (xy -2.196148 0.931115) (xy -2.47223 0.486614) (xy -2.653464 0.034691) (xy -2.746 -0.443079)
+				(xy -2.761528 -0.762) (xy -2.715952 -1.264644) (xy -2.584228 -1.749665) (xy -2.373866 -2.195886)
+				(xy -2.132409 -2.536425) (xy -2.038407 -2.640949) (xy -1.978828 -2.676911) (xy -1.923869 -2.65447)
+			)
+			(stroke
+				(width 0.01)
+				(type solid)
+			)
+			(fill solid)
+			(layer "F.SilkS")
+		)
+		(fp_poly
+			(pts
+				(xy 1.161168 -1.849741) (xy 1.239447 -1.782841) (xy 1.366292 -1.617475) (xy 1.480644 -1.385727)
+				(xy 1.567852 -1.122793) (xy 1.610772 -0.890985) (xy 1.600779 -0.564766) (xy 1.514239 -0.221701)
+				(xy 1.360921 0.101459) (xy 1.336848 0.1397) (xy 1.22659 0.287943) (xy 1.139439 0.347909) (xy 1.061514 0.325948)
+				(xy 1.020264 0.284538) (xy 0.995156 0.217867) (xy 1.027532 0.123569) (xy 1.087129 0.028039) (xy 1.227751 -0.225803)
+				(xy 1.300644 -0.488597) (xy 1.315186 -0.797431) (xy 1.312254 -0.862141) (xy 1.288982 -1.087307)
+				(xy 1.238808 -1.263503) (xy 1.145934 -1.442749) (xy 1.126104 -1.475109) (xy 1.036611 -1.625748)
+				(xy 0.997894 -1.718083) (xy 1.003402 -1.777693) (xy 1.037474 -1.821246) (xy 1.099352 -1.866702)
+				(xy 1.161168 -1.849741)
+			)
+			(stroke
+				(width 0.01)
+				(type solid)
+			)
+			(fill solid)
+			(layer "F.SilkS")
+		)
+		(fp_poly
+			(pts
+				(xy -2.735346 -3.461867) (xy -2.68835 -3.425335) (xy -2.646355 -3.379033) (xy -2.639155 -3.328849)
+				(xy -2.674835 -3.253934) (xy -2.76148 -3.133436) (xy -2.841559 -3.030246) (xy -3.165788 -2.543211)
+				(xy -3.418082 -1.99863) (xy -3.512 -1.72541) (xy -3.585816 -1.392648) (xy -3.625907 -1.001114) (xy -3.631741 -0.588061)
+				(xy -3.602786 -0.190744) (xy -3.538827 0.1524) (xy -3.383759 0.59512) (xy -3.162194 1.041533) (xy -2.896979 1.446947)
+				(xy -2.839165 1.521094) (xy -2.710685 1.687605) (xy -2.642773 1.797534) (xy -2.626601 1.868504)
+				(xy -2.644861 1.908928) (xy -2.712936 1.966124) (xy -2.786918 1.964903) (xy -2.880005 1.897358)
+				(xy -3.005398 1.755579) (xy -3.096551 1.6383) (xy -3.426565 1.141852) (xy -3.663962 0.638179) (xy -3.816673 0.105476)
+				(xy -3.89263 -0.47806) (xy -3.897519 -0.563608) (xy -3.881895 -1.192399) (xy -3.774078 -1.793624)
+				(xy -3.577071 -2.358456) (xy -3.293874 -2.878067) (xy -2.967117 -3.300495) (xy -2.857158 -3.417062)
+				(xy -2.78814 -3.467163) (xy -2.735346 -3.461867)
+			)
+			(stroke
+				(width 0.01)
+				(type solid)
+			)
+			(fill solid)
+			(layer "F.SilkS")
+		)
+		(fp_poly
+			(pts
+				(xy 2.031045 -2.606277) (xy 2.119837 -2.519352) (xy 2.159123 -2.474614) (xy 2.314165 -2.258078)
+				(xy 2.467092 -1.980955) (xy 2.598429 -1.682766) (xy 2.6887 -1.40303) (xy 2.69017 -1.397) (xy 2.752081 -0.966088)
+				(xy 2.742429 -0.512918) (xy 2.666355 -0.062063) (xy 2.528999 0.361903) (xy 2.335503 0.734407) (xy 2.208098 0.907158)
+				(xy 2.101656 1.021985) (xy 2.028574 1.060146) (xy 1.965286 1.029132) (xy 1.933567 0.994416) (xy 1.911346 0.936139)
+				(xy 1.935109 0.849845) (xy 2.012436 0.714043) (xy 2.056134 0.646956) (xy 2.176323 0.445977) (xy 2.289145 0.224787)
+				(xy 2.344162 0.09704) (xy 2.422175 -0.185791) (xy 2.46896 -0.522091) (xy 2.481522 -0.868273) (xy 2.456865 -1.180753)
+				(xy 2.438495 -1.275774) (xy 2.35734 -1.538426) (xy 2.238723 -1.820451) (xy 2.101112 -2.082847) (xy 1.962978 -2.286613)
+				(xy 1.955614 -2.295485) (xy 1.862014 -2.417301) (xy 1.835814 -2.496224) (xy 1.872754 -2.561386)
+				(xy 1.911644 -2.596315) (xy 1.96992 -2.627863) (xy 2.031045 -2.606277)
+			)
+			(stroke
+				(width 0.01)
+				(type solid)
+			)
+			(fill solid)
+			(layer "F.SilkS")
+		)
+		(fp_poly
+			(pts
+				(xy 2.896039 -3.371561) (xy 3.000333 -3.25402) (xy 3.338586 -2.785647) (xy 3.601411 -2.261549) (xy 3.785149 -1.697918)
+				(xy 3.88614 -1.110945) (xy 3.900726 -0.516819) (xy 3.825247 0.068269) (xy 3.787389 0.2286) (xy 3.691808 0.517398)
+				(xy 3.552313 0.840976) (xy 3.385655 1.16684) (xy 3.208585 1.462495) (xy 3.037854 1.69545) (xy 3.021375 1.7145)
+				(xy 2.883234 1.866436) (xy 2.791572 1.94905) (xy 2.728531 1.971648) (xy 2.676253 1.943541) (xy 2.645918 1.910203)
+				(xy 2.628781 1.857805) (xy 2.655357 1.77694) (xy 2.733789 1.650964) (xy 2.851013 1.491103) (xy 3.185907 0.982561)
+				(xy 3.423564 0.463654) (xy 3.568319 -0.078233) (xy 3.624509 -0.655717) (xy 3.625558 -0.762) (xy 3.577469 -1.362431)
+				(xy 3.438554 -1.933388) (xy 3.212606 -2.463939) (xy 2.903415 -2.943151) (xy 2.843134 -3.018379)
+				(xy 2.733633 -3.1546) (xy 2.681674 -3.238738) (xy 2.678932 -3.296065) (xy 2.717082 -3.351854) (xy 2.728917 -3.365086)
+				(xy 2.78378 -3.418247) (xy 2.83134 -3.423739) (xy 2.896039 -3.371561)
+			)
+			(stroke
+				(width 0.01)
+				(type solid)
+			)
+			(fill solid)
+			(layer "F.SilkS")
+		)
+		(fp_poly
+			(pts
+				(xy 0.255617 0.511349) (xy 0.381388 0.524331) (xy 0.447986 0.551348) (xy 0.476558 0.596801) (xy 0.476587 0.5969)
+				(xy 0.49682 0.668259) (xy 0.540331 0.823588) (xy 0.603236 1.048957) (xy 0.681651 1.330433) (xy 0.771691 1.654084)
+				(xy 0.862589 1.9812) (xy 0.960001 2.33161) (xy 1.049473 2.652817) (xy 1.12711 2.930888) (xy 1.189016 3.151893)
+				(xy 1.231297 3.301897) (xy 1.249601 3.3655) (xy 1.252237 3.393144) (xy 1.233437 3.414398) (xy 1.18175 3.430095)
+				(xy 1.085728 3.441067) (xy 0.93392 3.448151) (xy 0.714875 3.452178) (xy 0.417144 3.453983) (xy 0.029277 3.454399)
+				(xy 0.028823 3.4544) (xy -0.315151 3.452919) (xy -0.622812 3.448755) (xy -0.880441 3.442328) (xy -1.074323 3.434056)
+				(xy -1.190739 3.424357) (xy -1.218965 3.4163) (xy -1.204733 3.358558) (xy -1.165027 3.218213) (xy -1.104116 3.009809)
+				(xy -1.026269 2.747893) (xy -0.935756 2.447008) (xy -0.894651 2.3114) (xy -0.791626 1.971915) (xy -0.691253 1.640539)
+				(xy -0.599896 1.338329) (xy -0.523919 1.086344) (xy -0.469687 0.905643) (xy -0.460936 0.8763) (xy -0.351298 0.508)
+				(xy 0.049527 0.508) (xy 0.255617 0.511349)
+			)
+			(stroke
+				(width 0.01)
+				(type solid)
+			)
+			(fill solid)
+			(layer "F.SilkS")
 		)
 	)
